File: RPi-pHat-Thermocouple.sch (KiCad schematic (older format))
At the start: 37 parts, among them J1 RPi_GPIO, P1 CONN_01X02, P2 CONN_01X02, P3 CONN_01X02, P4 CONN_01X02, P6 CONN_01X03, Q1 NUD3124, SW1 Write, U1 MAX31850K, U2 DS18S20, U3 MAX31850K, U4 MAX31850K, U5 AT24CS32, U6 MAX31850K, U7 MCP1754ST

Commit message: Remove one MAX38150K add switching power supply
Removed one MAX38150K so now there are three on the board.
Added switching power supply to safely backpower the Raspberry Pi Zero.
Now has Barrel Jack for input power.
Updated schematic BOM fields and added KiBOM support.
Parts:
- removed C10, C14: 10nF, Capacitors_SMD:C_0603, symbol C_Small
- removed C9: 0.1uF, Capacitors_SMD:C_0603, symbol C_Small
- removed P4: CONN_01X02, Pin_Headers:Pin_Header_Straight_1x02_Pitch2.54mm, symbol CONN_01X02
- removed U6: MAX31850K, Housings_DFN_QFN_ML:TDFN-10-1EP_3x4mm_Pitch0.5mm, symbol MAX31850KATB
- added C12: 330uF, Capacitor_SMD:CP_Elec_10x7.9, symbol Device:CP_Small
- added C13, C17: 22uF, Capacitor_SMD:C_0805_2012Metric, symbol Device:C_Small
- added C14: 3300pF, Capacitor_SMD:C_0603_1608Metric, symbol Device:C_Small
- added D1, D2, D3: NUP2105LT1G, Package_TO_SOT_SMD:SOT-23, symbol Power_Protection-ML:NUP2105L
- added D4: (no value), Diode_SMD:Diode_Bridge_Vishay_DFS, symbol Device:D_Bridge_+-AA
- added FB1, FB2, FB3, FB4, FB5, FB6: 1k, Inductor_SMD:L_0603_1608Metric, symbol Device:Ferrite_Bead_Small
- added J2: Barrel_Jack_Switch, Connector_BarrelJack:BarrelJack_CUI_PJ-036AH-SMT_Horizontal, symbol Connector:Barrel_Jack_Switch
- added Q2: BCM857BS, Package_TO_SOT_SMD:SOT-363_SC-70-6, symbol Transistor_BJT-ML:BCM857BS
- added Q3: DMG2305UX, Package_TO_SOT_SMD:SOT-23, symbol Transistor_FET-ML:DMG2305UX
- added R6: 47k, Resistor_SMD:R_0603_1608Metric, symbol Device:R
- added R7: 10k, Resistor_SMD:R_0603_1608Metric, symbol Device:R
- added R8: 44.2k, Resistor_SMD:R_0603_1608Metric, symbol Device:R
- added R9: 232k, Resistor_SMD:R_0603_1608Metric, symbol Device:R
- added U6: LMZ21700, Converter_DCDC-ML:Converter_DCDC_Texas-SIL0008E, symbol Converter_DCDC-ML:LMZ21700
- BZ1: footprint cui-ml:CMI-9655S-SMT -> Buzzer_Beeper-ML:MagneticBuzzer_CUI-CMI-9655S; symbol CT-1205CL-SMT -> Device:Buzzer; Description (none) -> BUZ, SMD, 2.7kHz, 5V, 30mA
- C1, C4: footprint Capacitors_SMD:C_0603 -> Capacitor_SMD:C_0603_1608Metric; symbol C_Small -> Device:C_Small; Description (none) -> CAP, 0603, .1uF, 10%, X7R, 50V; Manufacturer Murata Electronics -> Yageo; Part Number GRM188R71H104KA93D -> CC0603KRX7R9BB104; Vendor Part Number 81-GRM39X104K50D -> 603-CC603KRX7R9BB104
- C10: renamed from C3; footprint Capacitors_SMD:C_0603 -> Capacitor_SMD:C_0603_1608Metric; symbol C_Small -> Device:C_Small; Description (none) -> CAP, 0603, .1uF, 10%, X7R, 50V; Manufacturer Murata Electronics -> Yageo; Part Number GRM188R71H104KA93D -> CC0603KRX7R9BB104; Vendor Part Number 81-GRM39X104K50D -> 603-CC603KRX7R9BB104
- C11: renamed from C7; footprint Capacitors_SMD:C_0603 -> Capacitor_SMD:C_0603_1608Metric; symbol C_Small -> Device:C_Small; Description (none) -> CAP, 0603, .1uF, 10%, X7R, 50V; Manufacturer Murata Electronics -> Yageo; Part Number GRM188R71H104KA93D -> CC0603KRX7R9BB104; Vendor Part Number 81-GRM39X104K50D -> 603-CC603KRX7R9BB104
- C15, C16: footprint Capacitors_SMD:C_0805 -> Capacitor_SMD:C_0805_2012Metric; symbol C_Small -> Device:C_Small; Description (none) -> CAP, 0805, 2.2uF, 10%, X7R, 16V; Manufacturer Murata Electronics -> Yageo; Part Number GRM21BR71C225KA12L -> CC0805KKX7R7BB225; Vendor Part Number 81-GRM21BR71C225KA2L -> 603-CC805KKX7R7BB225
- C2: renamed from C11; value 10nF -> 0.01uF; footprint Capacitors_SMD:C_0603 -> Capacitor_SMD:C_0603_1608Metric; symbol C_Small -> Device:C_Small; Description (none) -> CAP, 0603, .01uF, 10%, X7R, 50V; Part Number GRM188R71H103KA01D -> CC0603KRX7R9BB103; Vendor Part Number 81-GRM39X103K50D -> 603-CC603KRX7R9BB103
- C3: renamed from C2; value 10nF -> 0.1uF; footprint Capacitors_SMD:C_0603 -> Capacitor_SMD:C_0603_1608Metric; symbol C_Small -> Device:C_Small; Description (none) -> CAP, 0603, .1uF, 10%, X7R, 50V; Manufacturer Murata Electronics -> Yageo; Part Number GRM188R71H103KA01D -> CC0603KRX7R9BB104; Vendor Part Number 81-GRM39X103K50D -> 603-CC603KRX7R9BB104
- C5: renamed from C12; value 10nF -> 0.01uF; footprint Capacitors_SMD:C_0603 -> Capacitor_SMD:C_0603_1608Metric; symbol C_Small -> Device:C_Small; Description (none) -> CAP, 0603, .01uF, 10%, X7R, 50V; Part Number GRM188R71H103KA01D -> CC0603KRX7R9BB103; Vendor Part Number 81-GRM39X103K50D -> 603-CC603KRX7R9BB103
- C6: renamed from C5; value 10nF -> 0.1uF; footprint Capacitors_SMD:C_0603 -> Capacitor_SMD:C_0603_1608Metric; symbol C_Small -> Device:C_Small; Description (none) -> CAP, 0603, .1uF, 10%, X7R, 50V; Manufacturer Murata Electronics -> Yageo; Part Number GRM188R71H103KA01D -> CC0603KRX7R9BB104; Vendor Part Number 81-GRM39X103K50D -> 603-CC603KRX7R9BB104
- C7: renamed from C6; footprint Capacitors_SMD:C_0603 -> Capacitor_SMD:C_0603_1608Metric; symbol C_Small -> Device:C_Small; Description (none) -> CAP, 0603, .1uF, 10%, X7R, 50V; Manufacturer Murata Electronics -> Yageo; Part Number GRM188R71H104KA93D -> CC0603KRX7R9BB104; Vendor Part Number 81-GRM39X104K50D -> 603-CC603KRX7R9BB104
- C8: renamed from C13; value 10nF -> 0.01uF; footprint Capacitors_SMD:C_0603 -> Capacitor_SMD:C_0603_1608Metric; symbol C_Small -> Device:C_Small; Description (none) -> CAP, 0603, .01uF, 10%, X7R, 50V; Part Number GRM188R71H103KA01D -> CC0603KRX7R9BB103; Vendor Part Number 81-GRM39X103K50D -> 603-CC603KRX7R9BB103
- C9: renamed from C8; value 10nF -> 0.1uF; footprint Capacitors_SMD:C_0603 -> Capacitor_SMD:C_0603_1608Metric; symbol C_Small -> Device:C_Small; Description (none) -> CAP, 0603, .1uF, 10%, X7R, 50V; Manufacturer Murata Electronics -> Yageo; Part Number GRM188R71H103KA01D -> CC0603KRX7R9BB104; Vendor Part Number 81-GRM39X103K50D -> 603-CC603KRX7R9BB104
- J1: footprint raspberry-ml:Pin_Header_Straight_2x20 -> Connector_PinSocket_2.54mm:PinSocket_2x20_P2.54mm_Vertical; symbol RPi_GPIO -> Connector-ML:RPi_GPIO; Description (none) -> CON, THT, Dual Row Socket, 2.54mm, 40 Pos
- P1, P2, P3: symbol CONN_01X02 -> Connector_Generic:Conn_01x02; Description (none) -> CON, THT, Single Row, 2.54mm, 2 Pos, Pads; Notes (none) -> DNF
- P6: symbol CONN_01X03 -> Connector_Generic:Conn_01x03; Description (none) -> CON, THT, Single Row, 2.00mm, 3 Pos, Pads; Notes (none) -> DNF
- Q1: footprint TO_SOT_Packages_SMD:TSOT-23 -> Package_TO_SOT_SMD:SOT-23; symbol NUD3124 -> Power_Management-ML:NUD3124; Description (none) -> IC, SOT23, Inductive Load Driver
- R1, R5: footprint Resistors_SMD:R_0603 -> Resistor_SMD:R_0603_1608Metric; symbol R -> Device:R; Description (none) -> RES, 0603, 4.7k, 1%, T100
- R2, R3: footprint Resistors_SMD:R_0603 -> Resistor_SMD:R_0603_1608Metric; symbol R -> Device:R; Description (none) -> RES, 0603, 3.9k, 1%, T100
- R4: footprint Resistors_SMD:R_0603 -> Resistor_SMD:R_0603_1608Metric; symbol R -> Device:R; Description (none) -> RES, 0603, 1k, 1%, T100
- SW1: footprint Buttons_Switches_SMD:SW_SPST_B3U-3000P-B -> Button_Switch_SMD:SW_SPST_B3U-1000P; symbol SW_Push -> Switch:SW_Push; Description (none) -> SW, SMD, Push Button; Part Number B3U-3000P-B -> B3U-1000P; Vendor Part Number 653-B3U-3000P-B -> 653-B3U-1000P
- U1: footprint Housings_DFN_QFN_ML:TDFN-10-1EP_3x4mm_Pitch0.5mm -> Package_DFN_QFN-ML:TDFN-10-1EP_3x4mm_Pitch0.5mm; symbol MAX31850KATB -> Sensor_Temperature-ML:MAX31850KATB; Description (none) -> IC, TDFN10, 1-Wire Thermocouple Converter
- U2: renamed from U3; footprint Housings_DFN_QFN_ML:TDFN-10-1EP_3x4mm_Pitch0.5mm -> Package_DFN_QFN-ML:TDFN-10-1EP_3x4mm_Pitch0.5mm; symbol MAX31850KATB -> Sensor_Temperature-ML:MAX31850KATB; Description (none) -> IC, TDFN10, 1-Wire Thermocouple Converter
- U3: renamed from U4; footprint Housings_DFN_QFN_ML:TDFN-10-1EP_3x4mm_Pitch0.5mm -> Package_DFN_QFN-ML:TDFN-10-1EP_3x4mm_Pitch0.5mm; symbol MAX31850KATB -> Sensor_Temperature-ML:MAX31850KATB; Description (none) -> IC, TDFN10, 1-Wire Thermocouple Converter
- U4: renamed from U2; footprint TO_SOT_Packages_THT:TO-92_Molded_Narrow -> Package_TO_SOT_THT:TO-92; symbol DS18S20 -> Sensor_Temperature:DS18S20; Description (none) -> IC, TO92, 1-Wire Temperature Sensor
- U5: footprint Housings_SOIC:SOIC-8_3.9x4.9mm_Pitch1.27mm -> Package_DFN_QFN:DFN-8-1EP_3x2mm_P0.5mm_EP1.3x1.5mm; symbol AT24CS32-SSHM -> Memory_EEPROM-ML:AT24CS32-MAHM; Description (none) -> IC, DFN8, I2C Serial EEPROM, 32kbit; Part Number AT24CS32-SSHM -> AT24CS32-MAHM-E; Vendor Part Number 556-AT24CS32-SSHM-T -> 556-AT24CS32-MAHM-E
- U7: footprint TO_SOT_Packages_SMD:SOT89-3_Housing -> Package_TO_SOT_SMD:SOT-89-3; symbol MCP1754ST-3302E/MB -> Regulator_Linear:MCP1754-3302E_SOT89; Description (none) -> IC, SOT89-3, LDO VREG, 16V, .15A
Connections:
- net +3.3VA: now also C10.1, C11.1, R2.1, R3.1, R4.1, U4.3 (VDD), U5.8 (VCC); no longer C10.2
- net +5V: now also Q2.4 (E2), Q3.2 (S)
- net GND: now also C10.2, SW1.1, U4.1 (GND), C12.2, C13.2, C14.2, C17.2, D1.3 (A), D2.3 (A), D3.3 (A), D4.2 (-), R6.2, R7.2, R8.2, U6.10 (GND), U6.5 (GND), U6.9 (GND); no longer C10.1, SW1.2
- net TC1+: now also FB1.2; no longer C3.1, U1.3 (T+)
- net TC1-: now also FB2.2; no longer C3.2, U1.2 (T-)
- net TC2+: now also FB3.2; no longer C6.1, U2.3 (T+)
- net TC2-: now also FB4.2; no longer C6.2, U2.2 (T-)
- net TC3+: now also FB5.2; no longer C9.1, U3.3 (T+)
- net TC3-: now also FB6.2; no longer C9.2, U3.2 (T-)
- net W1: now also U4.2 (DQ)
- net at R4.2, U5.7 (WP): now also SW1.2; no longer SW1.1
- removed net +3V3: C11.1, J1.1 (3.3V), J1.17 (3.3V), R2.1, R3.1, R4.1, U5.8 (VCC)
- new net: C3.1, D1.1 (K), FB1.1, U1.3 (T+)
- new net: C3.2, D1.2 (K), FB2.1, U1.2 (T-)
- new net: C6.1, D2.1 (K), FB3.1, U2.3 (T+)
- new net: C6.2, D2.2 (K), FB4.1, U2.2 (T-)
- new net: C9.1, D3.1 (K), FB5.1, U3.3 (T+)
- new net: C9.2, D3.2 (K), FB6.1, U3.2 (T-)
- new net: C14.1, U6.1 (SS)
- new net: R8.1, R9.2, U6.2 (FB)
- new net: Q2.3 (C2), Q3.1 (G), R6.1
- new net: Q2.2 (B1), Q2.5 (B2), Q2.6 (C1), R7.1
- new net +5VB: C17.1, Q2.1 (E1), Q3.3 (D), R9.1, U6.4 (VOUT), U6.6 (VOS)
- new net AC1: D4.3 (~~), J2.1
- new net AC2: D4.4 (~~), J2.2
- new net VBulk: C12.1, C13.1, D4.1 (+), U6.7 (EN), U6.8 (VIN)
Other:
- note added: "1."
- note added: "5V Switcher"
- note added: "Ideal Diode"
- note added: "Maximum Raspberry Pi current is 650mA."
- note added: "Raspberry Pi Connector"
- note added: "Raspberry Pi can be safely back powered by this HAT."
- note added: "TC 1"
- note added: "TC 2"
- note added: "TC 3"
- note removed: "Thermocouple 1"
- note removed: "Thermocouple 2"
- note removed: "Thermocouple 3"
- note removed: "Thermocouple 4"
- moved on the sheet: BZ1, C1, C10, C11, C15, C16, C2, C3, C4, C5, C6, C7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
